Commit message: Add reorientation problem in pinocchio

File: src/multi_robot_multi_goal_planning/problems/urdfs/ur10e/ur10_spherized.urdf (robot description, URDF)
Before this commit: robot ur10e_robot, 11 links, 10 joints
Links:
- link forearm_link: geometry collision sphere radius=0.054763; collision sphere radius=0.062952
- link upper_arm_link: geometry collision sphere radius=0.070867; collision sphere radius=0.073298
- link wrist_3_link: geometry collision sphere radius=0.053571; collision sphere radius=0.063575
Joints:
- joint shoulder_lift_joint: limit lower=-6.283185307179586 upper=6.283185307179586 effort=330.0 velocity=2.0943951023931953 -> lower=-3.1415 upper=3.1415 effort=330.0 velocity=2.0943951023931953
- joint shoulder_pan_joint: limit lower=-6.283185307179586 upper=6.283185307179586 effort=330.0 velocity=2.0943951023931953 -> lower=-3.1415 upper=3.1415 effort=330.0 velocity=2.0943951023931953
- joint wrist_1_joint: limit lower=-6.283185307179586 upper=6.283185307179586 effort=56.0 velocity=3.141592653589793 -> lower=-3.1415 upper=3.1415 effort=56.0 velocity=3.141592653589793
- joint wrist_2_joint: limit lower=-6.283185307179586 upper=6.283185307179586 effort=56.0 velocity=3.141592653589793 -> lower=-3.1415 upper=3.1415 effort=56.0 velocity=3.141592653589793
- joint wrist_3_joint: limit lower=-6.283185307179586 upper=6.283185307179586 effort=56.0 velocity=3.141592653589793 -> lower=-3.1415 upper=3.1415 effort=56.0 velocity=3.141592653589793

Commit message: Move to relative paths for meshes

File: src/multi_robot_multi_goal_planning/problems/urdfs/ur10e/ur10_spherized.urdf (robot description, URDF)
Before this commit: robot ur10e_robot, 11 links, 10 joints
Links:
- link base_link_inertia: geometry collision sphere radius=0.113013; collision sphere radius=0.113017
- link forearm_link: geometry collision sphere radius=0.054763; collision sphere radius=0.062952
- link shoulder_link: geometry visual mesh filename=./shoulder.dae
- link upper_arm_link: geometry collision sphere radius=0.070867; collision sphere radius=0.073298
- link wrist_1_link: geometry visual mesh filename=./wrist1.dae
- link wrist_2_link: geometry collision sphere radius=0.05433; visual mesh filename=./wrist2.dae
- link wrist_3_link: geometry collision sphere radius=0.053571; collision sphere radius=0.063575

File: src/multi_robot_multi_goal_planning/problems/urdfs/ur5e/ur5e.urdf (robot description, URDF)
Before this commit: robot ur5e_robot, 11 links, 10 joints
Links:
- link base_link_inertia: geometry collision mesh filename=/home/valentin/git/postdoc/pin-venv/hello-world/ur5e_2nd_tr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; visual mesh filename=./base.dae
- link forearm_link: geometry collision mesh filename=/home/valentin/git/postdoc/pin-venv/hello-world/ur5e_2nd_tr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; visual mesh filename=./forearm.dae
- link shoulder_link: geometry collision mesh filename=/home/valentin/git/postdoc/pin-venv/hello-world/ur5e_2nd_tr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; visual mesh filename=./shoulder.dae
- link upper_arm_link: geometry collision mesh filename=/home/valentin/git/postdoc/pin-venv/hello-world/ur5e_2nd_tr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; visual mesh filename=./upperarm.dae
- link wrist_1_link: geometry collision mesh filename=/home/valentin/git/postdoc/pin-venv/hello-world/ur5e_2nd_tr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; visual mesh filename=./wrist1.dae
- link wrist_2_link: geometry collision mesh filename=/home/valentin/git/postdoc/pin-venv/hello-world/ur5e_2nd_tr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; visual mesh filename=./wrist2.dae
- link wrist_3_link: geometry collision mesh filename=/home/valentin/git/postdoc/pin-venv/hello-world/ur5e_2nd_tr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; visual mesh filename=./wrist3.dae

File: src/multi_robot_multi_goal_planning/problems/urdfs/ur5e/ur5e_constrained.urdf (robot description, URDF)
Before this commit: robot ur5e_robot, 11 links, 10 joints
Links:
- link base_link_inertia: geometry collision mesh filename=/home/valentin/git/postdoc/pin-venv/hello-world/ur5e_2nd_tr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; visual mesh filename=./base.dae
- link forearm_link: geometry collision mesh filename=/home/valentin/git/postdoc/pin-venv/hello-world/ur5e_2nd_tr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; visual mesh filename=./forearm.dae
- link shoulder_link: geometry collision mesh filename=/home/valentin/git/postdoc/pin-venv/hello-world/ur5e_2nd_tr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; visual mesh filename=./shoulder.dae
- link upper_arm_link: geometry collision mesh filename=/home/valentin/git/postdoc/pin-venv/hello-world/ur5e_2nd_tr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; visual mesh filename=./upperarm.dae
- link wrist_1_link: geometry collision mesh filename=/home/valentin/git/postdoc/pin-venv/hello-world/ur5e_2nd_tr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; visual mesh filename=./wrist1.dae
- link wrist_2_link: geometry collision mesh filename=/home/valentin/git/postdoc/pin-venv/hello-world/ur5e_2nd_tr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; visual mesh filename=./wrist2.dae
- link wrist_3_link: geometry collision mesh filename=/home/valentin/git/postdoc/pin-venv/hello-world/ur5e_2nd_tr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; visual mesh filename=./wrist3.dae
