Commit message: Update ur5 urdfs

File: src/multi_robot_multi_goal_planning/problems/urdfs/ur10e/ur10e_meshes.urdf (robot description, URDF)
Before this commit: robot ur10e_robot, 11 links, 10 joints
Links:
- link base_link_inertia: geometry collision mesh filename=./base.stl; visual mesh filename=./base.dae
- link forearm_link: geometry collision mesh filename=./forearm.stl; visual mesh filename=./forearm.dae
- link shoulder_link: geometry collision mesh filename=./shoulder.stl; visual mesh filename=./shoulder.dae
- link upper_arm_link: geometry collision mesh filename=./upperarm.stl; visual mesh filename=./upperarm.dae
- link wrist_1_link: geometry collision mesh filename=./wrist1.stl; visual mesh filename=./wrist1.dae
- link wrist_2_link: geometry collision mesh filename=./wrist2.stl; visual mesh filename=./wrist2.dae
- link wrist_3_link: geometry collision mesh filename=./wrist3.stl; visual mesh filename=./wrist3.dae

File: src/multi_robot_multi_goal_planning/problems/urdfs/ur10e/ur10e_primitives.urdf (robot description, URDF)
Before this commit: robot ur10e_robot, 11 links, 10 joints
Links:
- link base_link_inertia: geometry collision cylinder length=0.27 radius=0.08; visual mesh filename=./base.dae
- link forearm_link: geometry collision cylinder length=0.66 radius=0.06; visual mesh filename=./forearm.dae
- link shoulder_link: geometry visual mesh filename=./shoulder.dae
- link upper_arm_link: geometry collision cylinder length=0.71 radius=0.08; visual mesh filename=./upperarm.dae
- link wrist_1_link: geometry visual mesh filename=./wrist1.dae
- link wrist_2_link: geometry collision cylinder length=0.11 radius=0.05; visual mesh filename=./wrist2.dae
- link wrist_3_link: geometry collision cylinder length=0.15 radius=0.045; visual mesh filename=./wrist3.dae

File: src/multi_robot_multi_goal_planning/problems/urdfs/ur5e/ur5e.urdf (robot description, URDF)
Before this commit: robot ur5e_robot, 11 links, 10 joints
Links:
- link base_link_inertia: geometry collision mesh filename=./base.stl; visual mesh filename=./base.dae

File: src/multi_robot_multi_goal_planning/problems/urdfs/ur5e/ur5e_constrained.urdf (robot description, URDF)
Before this commit: robot ur5e_robot, 11 links, 10 joints
Links:
- link base_link_inertia: geometry collision mesh filename=./base.stl; visual mesh filename=./base.dae
- link forearm_link: geometry collision mesh filename=./forearm.stl; visual mesh filename=/home/valentin/git/postdoc/pin-venv/hello-world/ur5e_2nd_tr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
- link shoulder_link: geometry collision mesh filename=./shoulder.stl; visual mesh filename=./shoulder.dae
- link upper_arm_link: geometry collision mesh filename=./upperarm.stl; visual mesh filename=/home/valentin/git/postdoc/pin-venv/hello-world/ur5e_2nd_tr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
- link wrist_1_link: geometry collision mesh filename=./wrist1.stl; visual mesh filename=/home/valentin/git/postdoc/pin-venv/hello-world/ur5e_2nd_tr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
- link wrist_2_link: geometry collision mesh filename=./wrist2.stl; visual mesh filename=/home/valentin/git/postdoc/pin-venv/hello-world/ur5e_2nd_tr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
- link wrist_3_link: geometry collision mesh filename=./wrist3.stl; visual mesh filename=/home/valentin/git/postdoc/pin-venv/hello-world/ur5e_2nd_tr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

File: src/multi_robot_multi_goal_planning/problems/urdfs/ur5e/ur5e_constrained_coll_primitives.urdf (robot description, URDF)
Before this commit: robot ur5e_robot, 11 links, 10 joints
Links:
- link base_link_inertia: geometry collision cylinder length=0.1 radius=0.075; visual mesh filename=./base.dae
- link forearm_link: geometry collision cylinder length=0.45 radius=0.04; visual mesh filename=./forearm.dae
- link shoulder_link: geometry collision cylinder length=0.15 radius=0.06; visual mesh filename=./shoulder.dae
- link upper_arm_link: geometry collision cylinder length=0.53 radius=0.06; visual mesh filename=./upperarm.dae
- link wrist_1_link: geometry collision cylinder length=0.11 radius=0.04; visual mesh filename=./wrist1.dae
- link wrist_2_link: geometry collision cylinder length=0.1 radius=0.04; visual mesh filename=./wrist2.dae
- link wrist_3_link: geometry collision cylinder length=0.04 radius=0.04; visual mesh filename=./wrist3.dae
